File: esp_programmer.kicad_pcb (KiCad board)
At the start: 2 copper layers, 9 parts, among them J3 Conn_01x06_Pin, U1 AMS1117-3.3

Commit message: New push
Parts:
- moved D1 34.4 mm to (107.8, 67.5)
- moved I1 34.1 mm to (114.0, 60.2)
- moved R1 33.6 mm to (107.7, 65.0)
- moved RST1 33.2 mm to (123.0, 60.2)
- moved C2 33.2 mm to (107.7, 61.5)
- moved J3 32.4 mm to (103.5, 57.6)
- moved J1 32.0 mm to (136.0, 59.4)
- moved U1 31.8 mm to (118.5, 69.5)
- moved C1 22.8 mm to (107.7, 69.5), turned to 180 degrees
Connections:
- J1 pad 2: unconnected-(J1-Pin_2-Pad2) -> /tx2rx
- J1 pad 3: /I01 -> unconnected-(J1-Pin_3-Pad3)
- J1 pad 4: /rx2tx -> /3v3
- J1 pad 5: /tx2rx -> /I01
- J1 pad 6: /EN -> /rst
- J1 pad 7: /rst -> /rx2tx
Routing:
- net /3v3: track 0.00 -> 74.1 mm
- net /GND: track 0.00 -> 59.7 mm, vias 0 -> 2
- net /rx2tx: track 0.00 -> 51.6 mm
- net /tx2rx: track 0.00 -> 32.6 mm
- net /I01: track 0.00 -> 25.0 mm, vias 0 -> 1
- net /5V: track 0.00 -> 24.6 mm, vias 0 -> 1
- net /rst: track 0.00 -> 12.2 mm, vias 0 -> 1
- net /r1d1: track 0.00 -> 3.75 mm
Other:
- board outline added: 42 x 25 mm
